File: pcb/macropad.kicad_pcb (KiCad board)
At the start: 2 copper layers, 72.8 x 100 mm, 43 parts, among them SW1 SW_Push, SW10 SW_Push, SW11 SW_Push, SW12 SW_Push, SW13 RotaryEncoder_Switch, SW2 SW_Push, SW3 SW_Push, SW4 SW_Push, SW5 SW_Push, SW6 SW_Push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

Commit message: updating files
Connections:
- U1 pad 8: LED 2 -> LED 3
Routing:
- net LED 3: track 0.00 -> 113.8 mm
- net LED 2: track 42.4 -> 14.5 mm
Changed lines of the file:
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@@
 			(outputformat 1)
 			(mirror no)
-			(drillshape 1)
+			(drillshape 0)
 			(scaleselection 1)
-			(outputdirectory "")
+			(outputdirectory "gerbers/")
 		)
 	)
@@
 			(layers "*.Cu" "*.Mask")
 			(remove_unused_layers no)
-			(net 26 "LED 2")
+			(net 40 "LED 3")
 			(pinfunction "PB09_A7_D7_RX")
 			(pintype "passive")
@@
 	(segment
 		(start 212.0875 82.1)
-		(end 212.0875 75.5875)
-		(width 0.2)
-		(layer "B.Cu")
-		(net 26)
-	)
-	(segment
-		(start 200.5 64)
-		(end 195.55 64)
-		(width 0.2)
-		(layer "B.Cu")
-		(net 26)
-	)
-	(segment
-		(start 212.0875 82.1)
 		(end 212.8875 82.1)
 		(width 0.2)
@@
 	)
 	(segment
-		(start 212.0875 75.5875)
-		(end 200.5 64)
-		(width 0.2)
-		(layer "B.Cu")
-		(net 26)
-	)
-	(segment
-		(start 195.55 64)
-		(end 195.5 64.05)
-		(width 0.2)
-		(layer "B.Cu")
-		(net 26)
-	)
-	(segment
 		(start 203.139 117.389)
 		(end 203.139 104.361)
@@
 		(net 39)
 	)
+	(segment
+		(start 237.8 132.5875)
+		(end 237.8 75.15)
+		(width 0.2)
+		(layer "B.Cu")
+		(net 40)
+	)
+	(segment
+		(start 233.501 70.851)
+		(end 202.301 70.851)
+		(width 0.2)
+		(layer "B.Cu")
+		(net 40)
+	)
+	(segment
+		(start 237.8 75.15)
+		(end 233.501 70.851)
+		(width 0.2)
+		(layer "B.Cu")
+		(net 40)
+	)
+	(segment
+		(start 231.1375 139.25)
+		(end 237.8 132.5875)
+		(width 0.2)
+		(layer "B.Cu")
+		(net 40)
+	)
+	(segment
+		(start 202.301 70.851)
+		(end 195.5 64.05)
+		(width 0.2)
+		(layer "B.Cu")
+		(net 40)
+	)
+	(segment
+		(start 195.55 64)
+		(end 195.5 64.05)
+		(width 0.2)
+		(layer "B.Cu")
+		(net 40)
+	)
 	(embedded_fonts no)
